Commit message: src from 2.2.3 and gazebo plugins from master

File: rotors_description/urdf/component_snippets.xacro (robot description, xacro)
@@ -17,4 +17,5 @@
 -->
 <robot xmlns:xacro="http://ros.org/wiki/xacro">
+  <xacro:property name="pi" value="3.14159265359" />
   <!-- Macro to add logging to a bag file. -->
   <xacro:macro name="bag_plugin_macro"
